Commit message: updated launch and urdf for ldlidar and wheel joint names and  roboclaw.yaml to publish robot states

File: robots/stingray/description/ldlidar_support.xacro (robot description, xacro)
@@ -19,5 +19,5 @@
         <!-- Front standoff -->
         <visual name="ldlidar_support_front">
-            <origin xyz="${ldlidar_support_offset_x + 0.0234} ${ldlidar_support_offset_y} ${ldlidar_support_height/2}" rpy="0.0 0.0 0.0"/>
+            <origin xyz="${ldlidar_offset_x + 0.0234} ${ldlidar_offset_y} ${ldlidar_support_height/2}" rpy="0.0 0.0 0.0"/>
             <geometry>
                 <cylinder radius="0.003175" length="${ldlidar_support_height}"/>
@@ -27,5 +27,5 @@
         <!-- Right rear standoff -->
         <visual name="ldlidar_support_right">
-            <origin xyz="${ldlidar_support_offset_x - 0.00846} ${ldlidar_support_offset_y - 0.02333} ${ldlidar_support_height/2}" rpy="0.0 0.0 0.0"/>
+            <origin xyz="${ldlidar_offset_x - 0.00846} ${ldlidar_offset_y - 0.02333} ${ldlidar_support_height/2}" rpy="0.0 0.0 0.0"/>
             <geometry>
                 <cylinder radius="0.003175" length="${ldlidar_support_height}"/>
@@ -35,5 +35,5 @@
         <!-- Left rear standoff -->
         <visual name="ldlidar_support_left">
-            <origin xyz="${ldlidar_support_offset_x - 0.00846} ${ldlidar_support_offset_y + 0.02333} ${ldlidar_support_height/2}" rpy="0.0 0.0 0.0"/>
+            <origin xyz="${ldlidar_offset_x - 0.00846} ${ldlidar_offset_y + 0.02333} ${ldlidar_support_height/2}" rpy="0.0 0.0 0.0"/>
             <geometry>
                 <cylinder radius="0.003175" length="${ldlidar_support_height}"/>

File: robots/stingray/description/robot.urdf.xacro (robot description, xacro)
@@ -19,10 +19,10 @@
     <xacro:property name="imu_visual_size" value="0.01"/>
     <xacro:include filename="../../../description/imu.xacro" />
-    <xacro:property name="laser_offset_x" value="0.085"/>
-    <xacro:property name="laser_offset_z" value="0.033"/>
     <!-- Note: regular camera and depth camera share chassis' "camera_link". Use one or another.  -->
     <!-- xacro:include filename="stingray_camera.xacro" / -->
     <xacro:include filename="stingray_depth_camera.xacro" />
-    <xacro:include filename="stingray_lidar.urdf.xacro" />
+    <!-- LDLidar configuration - ldlidar must be included before support to define properties -->
+    <xacro:include filename="ldlidar.xacro" />
+    <xacro:include filename="ldlidar_support.xacro" />
     <xacro:include filename="ros2_control.xacro" />
     <xacro:property name="open_circuit_voltage" value="14.0"/>

File: robots/stingray/description/robot_core.xacro (robot description, xacro)
@@ -72,5 +72,5 @@
     </link>
     <!-- WHEEL LINKS -->
-    <joint name="wheel_left_joint" type="continuous">
+    <joint name="left_wheel_joint" type="continuous">
         <parent link="base_link"/>
         <child link="left_wheel_link"/>
@@ -101,5 +101,5 @@
         </xacro:inertial_cylinder>
     </link>
-    <joint name="wheel_right_joint" type="continuous">
+    <joint name="right_wheel_joint" type="continuous">
         <parent link="base_link"/>
         <child link="right_wheel_link"/>
