Commit message: Update ldlidar, lidar orientation, BNO085, IMU calibration orientation.

File: robots/stingray/description/BNOxxx_imu.xacro (robot description, xacro)
@@ -12,5 +12,4 @@
         <visual>
             <geometry>
-                <!-- <box size="0.1 0.1 0.1"/> -->
                 <box size="0.016 0.020 0.004"/>
             </geometry>

File: robots/stingray/description/ldlidar.xacro (robot description, xacro)
@@ -12,4 +12,5 @@
     <xacro:property name="ldlidar_rotation_x" value="0.0"/>
     <xacro:property name="ldlidar_rotation_y" value="0.0"/>
+    <!-- <xacro:property name="ldlidar_rotation_z" value="${-pi/2}"/> -->
     <xacro:property name="ldlidar_rotation_z" value="${-pi/2}"/>
     <joint name="ldlaser_joint" type="fixed">

File: robots/stingray/description/robot.urdf.xacro (robot description, xacro)
@@ -15,8 +15,13 @@
     <xacro:include filename="stingray_properties.xacro" />
     <xacro:include filename="robot_core.xacro" />
-    <xacro:property name="imu_offset_x" value="-0.04"/>
-    <xacro:property name="imu_offset_z" value="0"/>
-    <xacro:property name="imu_visual_size" value="0.01"/>
-    <xacro:include filename="../../../description/imu.xacro" />
+    <xacro:property name="imu_offset_x" value="0.0"/>
+    <xacro:property name="imu_offset_y" value="0.0"/>
+    <xacro:property name="imu_offset_z" value="0.0"/>
+    <xacro:property name="imu_rotation_x" value="0.0"/>
+    <xacro:property name="imu_rotation_y" value="0.0"/>
+    <xacro:property name="imu_rotation_z" value="0.0"/>
+    <!-- <xacro:property name="imu_visual_size" value="0.01"/> -->
+    <!-- <xacro:include filename="../../../description/BNOxxx_imu.xacro" /> -->
+    <xacro:include filename="BNOxxx_imu.xacro" />
     <!-- Note: regular camera and depth camera share chassis' "camera_link". Use one or another.  -->
     <!-- xacro:include filename="stingray_camera.xacro" / -->

File: robots/stingray/description/robot_core.xacro (robot description, xacro)
@@ -9,5 +9,5 @@
             <origin xyz="0 0 0"/>
             <geometry>
-                <sphere radius="0.01"/>
+                <sphere radius="0.005"/>
             </geometry>
             <material name="red"/>
