Commit message: added -0.60 imu_rotation_z to robot.urdf.xacro to fix IMU skew

File: robots/stingray/description/robot.urdf.xacro (robot description, xacro)
@@ -20,5 +20,6 @@
     <xacro:property name="imu_rotation_x" value="0.0"/>
     <xacro:property name="imu_rotation_y" value="0.0"/>
-    <xacro:property name="imu_rotation_z" value="0.0"/>
+    <!-- -35 degrees to correct IMU frame offset -->
+    <xacro:property name="imu_rotation_z" value="-0.6000"/>
     <!-- <xacro:property name="imu_visual_size" value="0.01"/> -->
     <!-- <xacro:include filename="../../../description/BNOxxx_imu.xacro" /> -->

Commit message: final imu_rotation_z

File: robots/stingray/description/robot.urdf.xacro (robot description, xacro)
@@ -21,5 +21,5 @@
     <xacro:property name="imu_rotation_y" value="0.0"/>
     <!-- -35 degrees to correct IMU frame offset -->
-    <xacro:property name="imu_rotation_z" value="-0.6000"/>
+    <xacro:property name="imu_rotation_z" value="-0.7048"/>
     <!-- <xacro:property name="imu_visual_size" value="0.01"/> -->
     <!-- <xacro:include filename="../../../description/BNOxxx_imu.xacro" /> -->

Commit message: fix base_footprint, IMU rotation (again)

File: robots/stingray/description/robot.urdf.xacro (robot description, xacro)
@@ -21,5 +21,5 @@
     <xacro:property name="imu_rotation_y" value="0.0"/>
     <!-- -35 degrees to correct IMU frame offset -->
-    <xacro:property name="imu_rotation_z" value="-0.7048"/>
+    <xacro:property name="imu_rotation_z" value="-0.7650"/>
     <!-- <xacro:property name="imu_visual_size" value="0.01"/> -->
     <!-- <xacro:include filename="../../../description/BNOxxx_imu.xacro" /> -->

File: robots/stingray/description/robot_core.xacro (robot description, xacro)
@@ -1,4 +1,5 @@
 ﻿<?xml version="1.0" encoding="UTF-8"?>
 <robot xmlns:xacro="http://ros.org/wiki/xacro">
+    <xacro:property name="oakd_x_length" value="0.033"/>
     <!-- BASE LINK -->
     <link name="base_link">
@@ -25,7 +26,7 @@
     <link name="base_footprint">
         <visual name="footprint_visual">
-            <origin xyz="-${chassis_offset + caster_radius} 0.0 0.0"/>
+            <origin xyz="-${chassis_offset + caster_radius - (oakd_x_length/2)} 0.0 0.0"/>
             <geometry>
-                <box size="${chassis_length + (caster_radius * 2)} ${wheel_separation + wheel_thickness} 0.001"/>
+                <box size="${chassis_length + (caster_radius * 2) + oakd_x_length} ${wheel_separation + wheel_thickness} 0.001"/>
             </geometry>
             <material name="shadow_gray"/>

Commit message: twist_mux, robot.urdf.xacro

File: robots/stingray/description/robot.urdf.xacro (robot description, xacro)
@@ -20,6 +20,5 @@
     <xacro:property name="imu_rotation_x" value="0.0"/>
     <xacro:property name="imu_rotation_y" value="0.0"/>
-    <!-- -35 degrees to correct IMU frame offset -->
-    <xacro:property name="imu_rotation_z" value="-0.7650"/>
+    <xacro:property name="imu_rotation_z" value="0.0"/>
     <!-- <xacro:property name="imu_visual_size" value="0.01"/> -->
     <!-- <xacro:include filename="../../../description/BNOxxx_imu.xacro" /> -->
