Commit message: make Gazebo lidar blue

File: robots/stingray/description/ldlidar.xacro (robot description, xacro)
@@ -52,5 +52,5 @@
     <link name="base_laser"/>
     <gazebo reference="ldlaser_frame">
-        <material>Gazebo/Grey</material>
+        <material>Gazebo/Blue</material>
     	    <sensor name="ldlaser_frame" type="gpu_lidar">
             <pose> 0.0 0.0 0.0 0.0 0.0 0.0 </pose>

Commit message: change ldlidar blue > black

File: robots/stingray/description/ldlidar.xacro (robot description, xacro)
@@ -25,5 +25,5 @@
                 <box size="${ldlidar_chassis_width} ${ldlidar_chassis_width} ${ldlidar_chassis_height}"/>
             </geometry>
-            <material name="blue"/>
+            <material name="black"/>
         </visual>
         <visual>
@@ -32,5 +32,5 @@
                 <cylinder radius="${ldlidar_radius}" length="${ldlidar_height}"/>
             </geometry>
-            <material name="blue"/>
+            <material name="black"/>
         </visual>
         <collision>
@@ -52,5 +52,5 @@
     <link name="base_laser"/>
     <gazebo reference="ldlaser_frame">
-        <material>Gazebo/Blue</material>
+        <material>Gazebo/Black</material>
     	    <sensor name="ldlaser_frame" type="gpu_lidar">
             <pose> 0.0 0.0 0.0 0.0 0.0 0.0 </pose>
