Commit message: stingray: fix OAK/lidar extrinsics, add hall-table keepout, lower OAK gate; diagnose low-obstacle marking
Low shelf (0.136-0.156 m) under the hall table never marks as a costmap
obstacle, so Stormy drives under it and hangs. Investigated live:

Root cause: OAK sees the shelf richly; points land in the correct in-grid
local voxel (iz=1) but Nav2's VoxelLayer never records a mark (voxel stays
UNKNOWN) while the taller wall marks fine. Ruled out clearing, height gate,
origin_z, resolution, mark_threshold (=0), and marking-only/max. The returns
are low/close/just-above-camera (near-horizontal) -- an ingestion/geometry
issue below the costmap parameter surface. No software knob reaches it.

Changes:
- robot.urdf.xacro: OAK mount pitch 0 -> 0.027 rad (~1.55 deg nose-down).
  Corrects screw-induced tilt; floor plane flattened ~1.4deg -> ~0.17deg
  (verified). Re-verify on clean floor.
- stingray_properties.xacro / ldlidar.xacro: chassis_height 0.081->0.0882,
  ldlidar_chassis_height 0.0228->0.022, scan-plane formula -> base_laser at
  0.1757 m (measured 0.1755; was ~8.6 mm low). E-stop/battery rise 3.6 mm (ok).
- assets/maps/keepout_mask.pgm: keepout rectangle over the hall table
  (map x[-1.12,0.0] y[1.50,2.19]); deterministic net, planner refuses it.
- nav2_params.yaml: global OAK min_obstacle_height 0.10 -> 0.06 (safe now that
  the floor is flat; catches low obstacles the layer does ingest).

Next: up-tilt the OAK (~1/2 vertical FOV) so low returns leave the degenerate
near-horizontal regime and mark honestly; add up-tilted sonar for glass. See
robots/stingray/NOTES-2026-10-03-low-obstacle-detection.md.

Co-authored-by: Copilot <223556219+Copilot@users.noreply.github.com>

File: robots/stingray/description/ldlidar.xacro (robot description, xacro)
@@ -4,5 +4,5 @@
     <xacro:property name="ldlidar_radius" value="0.017645"/>
     <xacro:property name="ldlidar_height" value="0.012"/>
-    <xacro:property name="ldlidar_chassis_height" value="0.0228"/>
+    <xacro:property name="ldlidar_chassis_height" value="0.022"/>
     <xacro:property name="ldlidar_chassis_width" value="0.038"/>
     <xacro:property name="ldlidar_support_height" value="0.0381"/>
@@ -48,5 +48,9 @@
         <parent link="ldlaser_frame"/>
         <child link="base_laser"/>
-        <origin xyz="0 0 ${ldlidar_chassis_height + ldlidar_height/2 - 0.0015}" rpy="0 0 0"/>
+        <!-- 2026-10-03: scan plane sits 2mm below the top of the 12mm LD19 body,
+             i.e. 0.010 m above the lidar base, so base + (height - 0.002) = 0.022 + 0.010
+             = 0.032. Full stack to floor now 0.0615+0.0441+0.0381+0.032 = 0.1757 m
+             (measured 0.1755). Was 0.0273 (~8mm low). -->
+        <origin xyz="0 0 ${ldlidar_chassis_height + ldlidar_height - 0.002}" rpy="0 0 0"/>
     </joint>
     <link name="base_laser"/>

File: robots/stingray/description/robot.urdf.xacro (robot description, xacro)
@@ -32,5 +32,13 @@
     <xacro:include filename="$(find articubot_one)/description/oakd.xacro" />
     <xacro:oakd_link mount_point="front_panel"/>
-    <xacro:oakd_joint x="0.023" y="0.01" z="0.030" roll="0" pitch="0" yaw="0" mount_point="front_panel"/>
+    <!-- 2026-10-03: pitch 0 -> 0.024 -> 0.027 rad (~1.55 deg nose-down). The anti-roll
+         mount screws tip the camera forward; the OAK floor plane was measured rising ~1.4
+         deg with range (drydock, level chassis) while the model assumed level, so the
+         costmap saw a sloped floor. 0.024 rad flattened it to a +0.17 deg residual (on
+         tile, table in far bins), so +0.17 deg -> 0.027 rad to zero it. Positive pitch =
+         nose-down (parent base_link, +x fwd). The 0.17 deg is within measurement noise
+         (~6 mm/2 m); re-verify with the floor-flatness probe on CLEAN floor (no table
+         ahead) and adjust until slope ~ 0 (flip sign if it worsens). -->
+    <xacro:oakd_joint x="0.023" y="0.01" z="0.030" roll="0" pitch="0.027" yaw="0" mount_point="front_panel"/>
     <!-- LDLidar configuration - ldlidar must be included before support to define properties -->
     <xacro:include filename="ldlidar.xacro" />

File: robots/stingray/description/stingray_properties.xacro (robot description, xacro)
@@ -3,5 +3,10 @@
     <xacro:property name="chassis_length" value="0.266"/>
     <xacro:property name="chassis_width" value="0.228"/>
-    <xacro:property name="chassis_height" value="0.081"/>
+    <!-- 2026-10-03: 0.081->0.0882. Real chassis = 3" (0.0762) side panels + 6mm top
+         + 6mm bottom plate = 0.0882, centered on base_link (side-panel centerline).
+         Makes chassis_height/2 = 0.0441 = base_link->chassis-top, which the lidar
+         support, e-stop and battery mounts rely on. Measured chassis top = 105mm off
+         floor = wheel_radius(0.0615) + 0.0441. -->
+    <xacro:property name="chassis_height" value="0.0882"/>
     <!--chassis_offset is distance from center of chassis
     to chassis origin between the wheels at base_link -->
