Commit message: make OAK-D appear in Gazebo and black in Gazebor and Rviz

File: description/oakd.xacro (robot description, xacro)
@@ -12,7 +12,9 @@
               <origin rpy="0 0 0" xyz="0 0 0" />
               <geometry>
-                      <mesh filename="package://articubot_one/assets/meshes/OAK-D.dae"/>
+                      <mesh filename="file://$(find articubot_one)/assets/meshes/OAK-D.dae"/>
               </geometry>
-               <material name="black" />
+               <material name="black">
+                   <color rgba="0.0 0.0 0.0 1.0"/>
+               </material>
           </visual>
           <collision>
@@ -60,5 +62,5 @@
   <!-- Gazebo plugin for greyscale left/right stereo pairs -->
       <gazebo reference="oakd_${mount_point}">
-    <material>Gazebo/Grey</material>
+    <material>Gazebo/Black</material>
     <sensor type="multicamera" name="stereo_camera">
       <update_rate>30.0</update_rate>
@@ -83,5 +85,5 @@
       <camera name="right">
         <pose>0 -0.07 0 0 0 0</pose>
-        <horizontal_fov>1.1.2566</horizontal_fov>
+        <horizontal_fov>1.2566</horizontal_fov>
         <image>
           <width>1200</width>
@@ -119,5 +121,5 @@
  <!-- Gazebo plugin for center RGB camera -->
    <gazebo reference="oakd_${mount_point}">
-      <material>Gazebo/White</material>
+      <material>Gazebo/Black</material>
       <sensor type="camera" name="oakd_rgb_${mount_point}">
       <update_rate>30.0</update_rate>

Commit message: URDF: use package:// mesh URIs so Foxglove can fetch them
Foxglove's asset bridge serves package:// but blocks file://. RViz/Gazebo
handle both, so this is a no-op for them and gains live model visualization
in Foxglove.

File: description/oakd.xacro (robot description, xacro)
@@ -12,5 +12,5 @@
               <origin rpy="0 0 0" xyz="0 0 0" />
               <geometry>
-                      <mesh filename="file://$(find articubot_one)/assets/meshes/OAK-D.dae"/>
+                      <mesh filename="package://articubot_one/assets/meshes/OAK-D.dae"/>
               </geometry>
                <material name="black">

File: robots/stingray/description/robot_core.xacro (robot description, xacro)
@@ -46,5 +46,5 @@
                 <!-- mesh filename="package://stingray/assets/meshes/Stingray.stl" scale="0.001 0.001 0.001"/-->
                 <!-- mesh filename="/home/ubuntu/stingray_ws/src/stingray/assets/meshes/Stingray.stl" scale="0.001 0.001 0.001"/-->
-                <mesh filename="file://$(find articubot_one)/assets/meshes/Stingray.stl" scale="0.001 0.001 0.001"/>
+                <mesh filename="package://articubot_one/assets/meshes/Stingray.stl" scale="0.001 0.001 0.001"/>
             </geometry>
             <material name="body_gray"/>
@@ -54,5 +54,5 @@
             <geometry>
                 <!-- box size="${chassis_length} ${chassis_width} ${chassis_height}"/ -->
-                <mesh filename="file://$(find articubot_one)/assets/meshes/Stingray.stl" scale="0.001 0.001 0.001"/>
+                <mesh filename="package://articubot_one/assets/meshes/Stingray.stl" scale="0.001 0.001 0.001"/>
                 <!-- mesh filename="/home/ubuntu/stingray_ws/src/stingray/assets/meshes/Stingray.stl" scale="0.001 0.001 0.001"/-->
                 <!-- mesh filename="file://home/ubuntu/stingray_ws/src/stingray/assets/meshes/Stingray.stl" scale="0.001 0.001 0.001"/-->
